File: PS-MPPTFanBoard.kicad_sch (KiCad schematic)
At the start: 30 parts, among them J1 Fan1, J10 Thermistor_Connecter, J2 Fan2, J3 Fan3, J4 Fan4, J7 CAN_NANO_02x05, J8 CAN_NANO_02x03, J9 CarLVPowerConnector

Commit message: not pretty
Parts:
- removed D17: FanStatus, LED_SMD:LED_0603_1608Metric_Pad1.05x0.95mm_HandSolder, symbol Device:LED
- removed R40: 120, Resistor_SMD:R_0603_1608Metric_Pad0.98x0.95mm_HandSolder, symbol Device:R_US
- removed R46: 10k, Resistor_SMD:R_0603_1608Metric_Pad0.98x0.95mm_HandSolder, symbol Device:R_US
- removed R47: 3.6, Resistor_SMD:R_0603_1608Metric_Pad0.98x0.95mm_HandSolder, symbol Device:R_US
- added R46: 10k, Resistor_SMD:R_0603_1608Metric_Pad0.98x0.95mm_HandSolder, symbol Device:R
- added R47: 3.6k, Resistor_SMD:R_0603_1608Metric_Pad0.98x0.95mm_HandSolder, symbol Device:R
- J7: value CAN_NANO_02x05 -> MPPT_CAN
- J8: value CAN_NANO_02x03 -> Car_CAN
- J9: value CarLVPowerConnector -> Car_Power
- R41, R42, R43, R49: value 120 -> 1k; symbol Device:R_US -> Device:R
- R44, R45: symbol Device:R_US -> Device:R
- R60: value 1k -> 4.7k; symbol Device:R_US -> Device:R
Connections:
- net 3.3V is gone; now on net +3.3V: R45.1
- net +12V: now also J1.1 (Pin_1), J2.1 (Pin_1), J3.1 (Pin_1), J4.1 (Pin_1), J7.1 (12V), J7.10 (12V)
- net GND: now also R47.2
- removed net 12V_Protected: J1.1 (Pin_1), J2.1 (Pin_1), J3.1 (Pin_1), J4.1 (Pin_1), J7.1 (12V), J7.10 (12V), J9.1 (+12V)
- new net 12V_In: J9.1 (+12V)
- new net 5V: R46.1
- new net Power_Mux/PR1: R46.2, R47.1
- no-connect marks 21 -> 22
Other:
- added sheet 12VBuck (12VBuck.kicad_sch)
- added sheet LDO (LDO.kicad_sch)
- added sheet Power_Mux (Power_Mux.kicad_sch)
- added sheet USB-C_Connector (USB-C_Connector.kicad_sch)
- moved on the sheet: D19, D23, D24, D25, H5, H6, H7, H8, J1, J10, J2, J3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
