File: PS-MPPTFanBoard.kicad_sch (KiCad schematic)
At the start: 27 parts, among them J1 Fan 1, 2, J10 Thermistor_Connecter, J2 Fan 3, 4, J7 MPPT_CAN, J8 Car_CAN, J9 Car_Power

Commit message: layout reviews
Parts:
- removed J1: Fan 1, 2, LHRS_Connectors:Molex_Nano-Fit_105310-xx06_2x03_P2.50mm_Vertical, symbol Connector_Generic:Conn_02x03_Counter_Clockwise
- removed J2: Fan 3, 4, LHRS_Connectors:Molex_Nano-Fit_105310-xx06_2x03_P2.50mm_Vertical, symbol Connector_Generic:Conn_02x03_Counter_Clockwise
- added F1: Fuse_3557_2, LHRS_Power:Fuse-3557-2, symbol lhrs_power:Fuse_3557_2
- added J1: Fan 1, 2, symbol Connector_Generic:Conn_02x04_Counter_Clockwise
- added J2: Fan 3, 4, symbol Connector_Generic:Conn_02x04_Counter_Clockwise
- D23: value Debug1 -> 5V
- D24: value Debug2 -> 3.3V
- R47: value 3.6k -> 4.7k
Connections:
- net +12V: now also J1.1 (Pin_1), J1.2 (Pin_2), J2.1 (Pin_1), J2.2 (Pin_2)
- net +3.3V: now also D24.2 (A)
- net +5V: now also D23.2 (A)
- net 12V_In: now also F1.2; no longer J9.1 (+12V)
- net DEBUG1: no longer D23.2 (A)
- net DEBUG2: no longer D24.2 (A)
- net FAN1_PWM: now also J1.6 (Pin_6)
- net FAN1_TACH: now also J1.3 (Pin_3)
- net FAN2_PWM: now also J1.5 (Pin_5)
- net FAN2_TACH: now also J1.4 (Pin_4)
- net FAN3_PWM: now also J2.6 (Pin_6)
- net FAN3_TACH: now also J2.3 (Pin_3)
- net FAN4_PWM: now also J2.5 (Pin_5)
- net FAN4_TACH: now also J2.4 (Pin_4)
- net GND: now also J1.7 (Pin_7), J1.8 (Pin_8), J2.7 (Pin_7), J2.8 (Pin_8)
- new net: F1.1, J9.1 (+12V)
