File: PS-MPPTFanBoard.kicad_sch (KiCad schematic)
At the start: 28 parts, among them J1 Fan 1, 2, J10 Thermistor_Connecter, J2 Fan 3, 4, J7 MPPT_CAN, J8 Car_CAN, J9 Car_Power

Commit message: gerbers and bom
Parts:
- J1, J2: P/N (none) -> 105310-1108
- J10: P/N (none) -> 105309-1102
Changed lines of the file:
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@@
 			)
 		)
+		(property "P/N" "105309-1102"
+			(at 227.33 57.15 0)
+			(hide yes)
+			(show_name no)
+			(do_not_autoplace no)
+			(effects
+				(font
+					(size 1.27 1.27)
+				)
+			)
+		)
 		(pin "2"
 		)
@@
 			)
 		)
+		(property "P/N" "105310-1108"
+			(at 33.02 130.81 0)
+			(hide yes)
+			(show_name no)
+			(do_not_autoplace no)
+			(effects
+				(font
+					(size 1.27 1.27)
+				)
+			)
+		)
 		(pin "7"
 		)
@@
 			(at 33.02 101.6 0)
 			(hide yes)
+			(show_name no)
+			(do_not_autoplace no)
+			(effects
+				(font
+					(size 1.27 1.27)
+				)
+			)
+		)
+		(property "P/N" "105310-1108"
+			(at 33.02 101.6 0)
+			(hide yes)
