File: 12VBuck.kicad_sch (KiCad schematic)
At the start: 10 parts, among them U4 LMR51635XDDCR

Commit message: layout placing
Parts:
- U4: footprint DDC0006A-MFG -> LHRS_ICs:DDC0006A-MFG
Changed lines of the file:
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@@
 			)
 		)
-		(property "Footprint" "DDC0006A-MFG"
+		(property "Footprint" "LHRS_ICs:DDC0006A-MFG"
 			(at 114.3 81.28 0)
 			(hide yes)
