File: USB-C_Connector.kicad_sch (KiCad schematic)
At the start: 4 parts, among them J11 USB_C_Receptacle_USB2.0_16P

Commit message: layout placing
Parts:
- J11: footprint LHRS_ICs:USB_C_Receptacle_GCT_USB4105-xx-A_16P_TopMnt_Horizontal -> LHRS_Connectors:USB_C_Receptacle_GCT_USB4105-xx-A_16P_TopMnt_Horizontal
Connections:
- net CC1: no longer names the net of J11.A5 (CC1)
- net CC2: no longer names the net of J11.B5 (CC2)
- no-connect marks 2 -> 4
Changed lines of the file:
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@@
+	)
+	(no_connect
+		(at 52.07 38.1)
 	)
 	(no_connect
@@
 	(no_connect
 		(at 50.8 58.42)
+	)
+	(no_connect
+		(at 52.07 35.56)
 	)
 	(wire
@@
 		)
 	)
-	(hierarchical_label "CC2"
-		(shape bidirectional)
-		(at 52.07 38.1 0)
-		(effects
-			(font
-				(size 1.27 1.27)
-			)
-			(justify left)
-		)
-	)
 	(hierarchical_label "USB_D-"
 		(shape bidirectional)
 		(at 55.88 44.45 0)
-		(effects
-			(font
-				(size 1.27 1.27)
-			)
-			(justify left)
-		)
-	)
-	(hierarchical_label "CC1"
-		(shape bidirectional)
-		(at 52.07 35.56 0)
 		(effects
 			(font
@@
 			)
 		)
-		(property "Footprint" "LHRS_ICs:USB_C_Receptacle_GCT_USB4105-xx-A_16P_TopMnt_Horizontal"
+		(property "Footprint" "LHRS_Connectors:USB_C_Receptacle_GCT_USB4105-xx-A_16P_TopMnt_Horizontal"
 			(at 39.37 45.72 0)
 			(hide yes)
