File: PS-MPPTFanBoard.kicad_pcb (KiCad board)
At the start: 2 copper layers, 100 x 49 mm, 139 parts, among them IC1 TCAN3413DR, IC2 LM74502DDFR, IC3 TCAN3413DR, J1 Fan 1, 2, J11 USB_C_Receptacle_USB2.0_16P, J2 Fan 3, 4, J5 SWD_Header, J6 SWD, Q1 PSMN012-100YS, Q2 PSMN012-100YS, SW1 Reset, SW2 SW_SPDT, U1 EMC2305-1-AP-TR, U2 STM32G473CETx, U3 MCP1826S, U4 LMR51635XDDCR, U5 TPS2117DRLR, Y1 Crystal

Commit message: finish
Routing:
- net /FAN_SDA: track 74.1 -> 71.8 mm
- net /FAN_SCL: track 72.0 -> 71.1 mm
- net +3.3V: track 247.4 -> 248.2 mm
- net /MPPT_CAN_RX: track 24.7 -> 25.5 mm
- net /~{SMBALERT}: track 85.1 -> 84.5 mm
- net GND: vias 63 -> 64
