File: Fans.kicad_sch (KiCad schematic)
At the start: 16 parts, among them U1 EMC2305-1-AP-TR

Commit message: not pretty
Parts:
- R12, R13, R16, R17, R18, R19, R20, R21, R6: symbol Device:R_US -> Device:R
Changed lines of the file:
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@@
 	)
 	(symbol
-		(lib_id "Device:R_US")
+		(lib_id "Device:R")
 		(at 228.6 58.42 180)
 		(unit 1)
@@
 		)
 		(property "Footprint" "Resistor_SMD:R_0603_1608Metric_Pad0.98x0.95mm_HandSolder"
-			(at 227.584 58.166 90)
+			(at 230.378 58.42 90)
 			(hide yes)
 			(show_name no)
@@
 			)
 		)
-		(property "Description" "Resistor, US symbol"
+		(property "Description" "Resistor"
 			(at 228.6 58.42 0)
 			(hide yes)
@@
 	)
 	(symbol
-		(lib_id "Device:R_US")
+		(lib_id "Device:R")
 		(at 254 58.42 180)
 		(unit 1)
@@
 		)
 		(property "Footprint" "Resistor_SMD:R_0603_1608Metric_Pad0.98x0.95mm_HandSolder"
-			(at 252.984 58.166 90)
+			(at 255.778 58.42 90)
 			(hide yes)
 			(show_name no)
@@
 			)
 		)
-		(property "Description" "Resistor, US symbol"
+		(property "Description" "Resistor"
 			(at 254 58.42 0)
 			(hide yes)
@@
 	)
 	(symbol
-		(lib_id "Device:R_US")
+		(lib_id "Device:R")
 		(at 173.99 35.56 180)
 		(unit 1)
@@
 		)
 		(property "Footprint" "Resistor_SMD:R_0603_1608Metric_Pad0.98x0.95mm_HandSolder"
-			(at 172.974 35.306 90)
+			(at 175.768 35.56 90)
 			(hide yes)
 			(show_name no)
@@
 			)
 		)
-		(property "Description" "Resistor, US symbol"
+		(property "Description" "Resistor"
 			(at 173.99 35.56 0)
 			(hide yes)
@@
 	)
 	(symbol
-		(lib_id "Device:R_US")
+		(lib_id "Device:R")
 		(at 173.99 58.42 180)
 		(unit 1)
@@
 		)
 		(property "Footprint" "Resistor_SMD:R_0603_1608Metric_Pad0.98x0.95mm_HandSolder"
-			(at 172.974 58.166 90)
+			(at 175.768 58.42 90)
 			(hide yes)
 			(show_name no)
@@
 			)
 		)
-		(property "Description" "Resistor, US symbol"
+		(property "Description" "Resistor"
 			(at 173.99 58.42 0)
 			(hide yes)
@@
 	)
 	(symbol
-		(lib_id "Device:R_US")
+		(lib_id "Device:R")
 		(at 44.45 36.83 180)
 		(unit 1)
@@
 		)
 		(property "Footprint" "Resistor_SMD:R_0603_1608Metric_Pad0.98x0.95mm_HandSolder"
-			(at 43.434 36.576 90)
+			(at 46.228 36.83 90)
 			(hide yes)
 			(show_name no)
@@
 			)
 		)
-		(property "Description" "Resistor, US symbol"
+		(property "Description" "Resistor"
 			(at 44.45 36.83 0)
 			(hide yes)
@@
 	)
 	(symbol
-		(lib_id "Device:R_US")
+		(lib_id "Device:R")
 		(at 255.27 35.56 180)
 		(unit 1)
@@
 		)
 		(property "Footprint" "Resistor_SMD:R_0603_1608Metric_Pad0.98x0.95mm_HandSolder"
-			(at 254.254 35.306 90)
+			(at 257.048 35.56 90)
 			(hide yes)
 			(show_name no)
@@
 			)
 		)
-		(property "Description" "Resistor, US symbol"
+		(property "Description" "Resistor"
 			(at 255.27 35.56 0)
 			(hide yes)
@@
 	)
 	(symbol
-		(lib_id "Device:R_US")
+		(lib_id "Device:R")
 		(at 228.6 35.56 180)
 		(unit 1)
@@
 		)
 		(property "Footprint" "Resistor_SMD:R_0603_1608Metric_Pad0.98x0.95mm_HandSolder"
-			(at 227.584 35.306 90)
+			(at 230.378 35.56 90)
 			(hide yes)
 			(show_name no)
@@
 			)
 		)
-		(property "Description" "Resistor, US symbol"
+		(property "Description" "Resistor"
 			(at 228.6 35.56 0)
 			(hide yes)
@@
 	)
 	(symbol
-		(lib_id "Device:R_US")
+		(lib_id "Device:R")
 		(at 64.77 34.29 180)
 		(unit 1)
@@
 		)
 		(property "Footprint" "Resistor_SMD:R_0603_1608Metric_Pad0.98x0.95mm_HandSolder"
-			(at 63.754 34.036 90)
+			(at 66.548 34.29 90)
 			(hide yes)
 			(show_name no)
@@
 			)
 		)
-		(property "Description" "Resistor, US symbol"
+		(property "Description" "Resistor"
 			(at 64.77 34.29 0)
 			(hide yes)
@@
 	)
 	(symbol
-		(lib_id "Device:R_US")
+		(lib_id "Device:R")
 		(at 134.62 45.72 180)
 		(unit 1)
@@
 		)
 		(property "Footprint" "Resistor_SMD:R_0603_1608Metric_Pad0.98x0.95mm_HandSolder"
-			(at 133.604 45.466 90)
+			(at 136.398 45.72 90)
 			(hide yes)
 			(show_name no)
@@
 			)
 		)
-		(property "Description" "Resistor, US symbol"
+		(property "Description" "Resistor"
 			(at 134.62 45.72 0)
 			(hide yes)

Commit message: layout placing
Parts:
- D16, D20, D21, D22: footprint UTSVT_Passive:SODFL5026X125N -> LHRS_Passives:SODFL5026X125N
- U1: footprint PumpLib:QFN16_4x4MC_MCH -> fanboard:QFN16_4x4MC_MCH
Connections:
- net 12V_Protected renamed +12V
Other:
- moved on the sheet: D16, D20, D21, D22

Commit message: gerbers and bom
Parts:
- D16, D20, D21, D22: P/N (none) -> VSSAF522-M3/H
- R12, R13, R6: P/N (none) -> CRCW06031K00FKEI
- R16, R17: P/N (none) -> 0603WAF3302TDE
- R18, R19, R20, R21: P/N (none) -> CRCW06035K10FKEC
Changed lines of the file:
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@@
+			)
+		)
+		(property "P/N" "VSSAF522-M3/H"
+			(at 35.56 101.6 90)
+			(hide yes)
+			(show_name no)
+			(do_not_autoplace no)
+			(effects
+				(font
+					(size 1.27 1.27)
+				)
 			)
 		)
@@
 			)
 		)
+		(property "P/N" "CRCW06035K10FKEC"
+			(at 228.6 58.42 0)
+			(hide yes)
+			(show_name no)
+			(do_not_autoplace no)
+			(effects
+				(font
+					(size 1.27 1.27)
+				)
+			)
+		)
 		(pin "2"
 		)
@@
 			)
 		)
+		(property "P/N" "CRCW06035K10FKEC"
+			(at 254 58.42 0)
+			(hide yes)
+			(show_name no)
+			(do_not_autoplace no)
+			(effects
+				(font
+					(size 1.27 1.27)
+				)
+			)
+		)
 		(pin "2"
 		)
@@
 			)
 		)
+		(property "P/N" "0603WAF3302TDE"
+			(at 173.99 35.56 0)
+			(hide yes)
+			(show_name no)
+			(do_not_autoplace no)
+			(effects
+				(font
+					(size 1.27 1.27)
+				)
+			)
+		)
 		(pin "2"
 		)
@@
 			)
 		)
+		(property "P/N" "VSSAF522-M3/H"
+			(at 54.61 101.6 90)
+			(hide yes)
+			(show_name no)
+			(do_not_autoplace no)
+			(effects
+				(font
+					(size 1.27 1.27)
+				)
+			)
+		)
 		(pin "1"
 		)
@@
 			)
 		)
+		(property "P/N" "0603WAF3302TDE"
+			(at 173.99 58.42 0)
+			(hide yes)
+			(show_name no)
+			(do_not_autoplace no)
+			(effects
+				(font
+					(size 1.27 1.27)
+				)
+			)
+		)
 		(pin "2"
 		)
@@
 			)
 		)
+		(property "P/N" "CRCW06031K00FKEI"
+			(at 44.45 36.83 0)
+			(hide yes)
+			(show_name no)
+			(do_not_autoplace no)
+			(effects
+				(font
+					(size 1.27 1.27)
+				)
+			)
+		)
 		(pin "2"
 		)
@@
 			)
 		)
+		(property "P/N" "CRCW06035K10FKEC"
+			(at 255.27 35.56 0)
+			(hide yes)
+			(show_name no)
+			(do_not_autoplace no)
+			(effects
+				(font
+					(size 1.27 1.27)
+				)
+			)
+		)
 		(pin "2"
 		)
@@
 			)
 		)
+		(property "P/N" "CRCW06035K10FKEC"
+			(at 228.6 35.56 0)
+			(hide yes)
+			(show_name no)
+			(do_not_autoplace no)
+			(effects
+				(font
+					(size 1.27 1.27)
+				)
+			)
+		)
 		(pin "2"
 		)
@@
 			)
 		)
+		(property "P/N" "CRCW06031K00FKEI"
+			(at 64.77 34.29 0)
+			(hide yes)
+			(show_name no)
+			(do_not_autoplace no)
+			(effects
+				(font
+					(size 1.27 1.27)
+				)
+			)
+		)
 		(pin "2"
 		)
@@
 		(property "Description" "1700V, 25A, SiC Schottky Diode, TO-247"
 			(at 73.66 101.6 0)
+			(hide yes)
+			(show_name no)
+			(do_not_autoplace no)
+			(effects
+				(font
+					(size 1.27 1.27)
+				)
+			)
+		)
+		(property "P/N" "VSSAF522-M3/H"
+			(at 73.66 101.6 90)
 			(hide yes)
 			(show_name no)
@@
 			)
 		)
+		(property "P/N" "CRCW06031K00FKEI"
+			(at 134.62 45.72 0)
+			(hide yes)
+			(show_name no)
+			(do_not_autoplace no)
+			(effects
+				(font
+					(size 1.27 1.27)
+				)
+			)
+		)
 		(pin "2"
 		)
@@
 			(hide yes)
 			(show_name no)
+			(do_not_autoplace no)
+			(effects
+				(font
+					(size 1.27 1.27)
+				)
+			)
+		)
+		(property "P/N" "VSSAF522-M3/H"
+			(at 92.71 101.6 90)
+			(hide yes)
+			(show_name no)
