File: LDO.kicad_sch (KiCad schematic)
At the start: 4 parts, among them U3 MCP1826S

Commit message: gerbers and bom
Parts:
- C33, C34: P/N (none) -> GRM21BR61H106KE43L
- D8: Old LCSC P/N C124187 -> (none); Old P/N BAT760-7 -> (none)
Changed lines of the file:
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@@
+			)
+		)
+		(property "P/N" "GRM21BR61H106KE43L"
+			(at 165.1 69.85 0)
+			(hide yes)
+			(show_name no)
+			(do_not_autoplace no)
+			(effects
+				(font
+					(size 1.27 1.27)
+				)
 			)
 		)
@@
 			)
 		)
-		(property "Old P/N" "BAT760-7"
-			(at 133.35 63.5 0)
-			(hide yes)
-			(show_name no)
-			(do_not_autoplace no)
-			(effects
-				(font
-					(size 1.27 1.27)
-				)
-			)
-		)
-		(property "Old LCSC P/N" "C124187"
-			(at 133.35 63.5 0)
-			(hide yes)
-			(show_name no)
-			(do_not_autoplace no)
-			(effects
-				(font
-					(size 1.27 1.27)
-				)
-			)
-		)
 		(pin "1"
 		)
@@
 			(at 139.7 69.85 0)
 			(hide yes)
+			(show_name no)
+			(do_not_autoplace no)
+			(effects
+				(font
+					(size 1.27 1.27)
+				)
+			)
+		)
+		(property "P/N" "GRM21BR61H106KE43L"
+			(at 139.7 69.85 0)
+			(hide yes)
