File: PowerProtection.kicad_sch (KiCad schematic)
At the start: 18 parts, among them IC2 LM74502DDFR, Q1 PSMN012-100YS, Q2 PSMN012-100YS

Commit message: gerbers and bom
Parts:
- R1: P/N 0603WAF1002T5E -> CRCW06031K00FKEI
Changed lines of the file:
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@@
 			)
 		)
-		(property "P/N" "0603WAF1002T5E"
+		(property "P/N" "CRCW06031K00FKEI"
 			(at 43.18 62.23 0)
 			(hide yes)
